Commit message: Change name: ros2_ to r3m_ObjectPoseEstimation (R3M Project).

File: ros2_opecalibration/urdf/calibenv.urdf.xacro (robot description, xacro)
@@ -36,5 +36,5 @@
       <origin xyz="0.0 0.0 0.0" rpy="0 0 0" />
       <geometry>
-        <mesh filename="file://$(find ros2_opecalibration)/meshes/objects/chessboard.dae" scale="1 1 1" />
+        <mesh filename="file://$(find r3m_opecalibration)/meshes/objects/chessboard.dae" scale="1 1 1" />
       </geometry>
     </visual>
@@ -42,5 +42,5 @@
       <origin xyz="0.0 0.0 0.0" rpy="0 0 0" />
       <geometry>
-        <mesh filename="file://$(find ros2_opecalibration)/meshes/objects/chessboard.dae" scale="1 1 1" />
+        <mesh filename="file://$(find r3m_opecalibration)/meshes/objects/chessboard.dae" scale="1 1 1" />
       </geometry>
     </collision>

File: ros2_opecalibration/urdf/objects/chessboard.urdf (robot description, URDF)
Before this commit: robot chessboard, 1 links, 0 joints
Links:
- link ${name}: geometry collision mesh filename=file://$(find r3m_ope)/meshes/objects/${name}.dae; visual mesh filename=file://$(find r3m_ope)/meshes/objects/${name}.dae
